File: UsbCanAdapter.kicad_pcb (KiCad board)
At the start: 2 copper layers, 57.4 x 31.1 mm, 32 parts, among them J1 Screw_Terminal_01x04, J2 USB_C_Receptacle_USB2.0, J3 SWD Pads, SW1 SW_Push, U1 STM32F042C6Tx, U3 MCP1700x-330xxTT

Commit message: Update PCB design for rev2 changes
Parts:
- added R6: 5.1k, Resistor_SMD:R_0603_1608Metric, F.Cu at (182.7, 68.0)
- moved C1 3.03 mm to (182.8, 72.0)
Connections:
- SW1 pad 1: GND1 -> VCC
Routing:
- net VCC: track 51.3 -> 59.3 mm, vias 1 -> 3
- net /BOOT0: track 17.3 -> 22.9 mm
- net GND1: track 43.8 -> 40.4 mm
- net /NRST: track 18.1 -> 16.3 mm
Other:
- board text added: "RJMP CAN Adapter REV 2"
- board text removed: "RJMP CAN Adapter REV 1"
